File: sandwichlamp.kicad_pcb (KiCad board)
At the start: 2 copper layers, 96 x 96 mm, 27 parts, among them J1 Pole1, J2 Pole2, J3 Pole3, J4 12V Enable, J5 HLK-LD2410C, J6 Conn_01x02, J7 Conn_01x03, SW1 Rader Power, SW3 POWER, U1 magnetic-charger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

Commit message: Run DRC
Connections:
- U7 pad 37: (no net) -> +4V
Routing:
- net GND: track 290.7 -> 312.1 mm
Changed lines of the file:
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@@
 			(at 0 -4.2 0)
 			(layer "F.SilkS")
+			(hide yes)
 			(effects
 				(font
@@
 		)
 		(fp_text user "+"
-			(at 6 -1.5 30)
+			(at 6.085641 -2.260639 30)
 			(unlocked yes)
 			(layer "B.Cu" knockout)
@@
 		(pad "1" thru_hole oval
 			(at -0.000001 -3.810001 90)
-			(size 2.3 3.2)
+			(size 1.7 3.2)
 			(drill 0.8
 				(offset 0 -0.4)
@@
 		(pad "2" thru_hole oval
 			(at 0 -1.270001 90)
-			(size 2.3 3.2)
+			(size 1.7 3.2)
 			(drill 0.8
 				(offset 0 -0.4)
@@
 		(pad "3" thru_hole oval
 			(at 0 1.270001 90)
-			(size 2.3 3.2)
+			(size 1.7 3.2)
 			(drill 0.8
 				(offset 0 -0.4)
@@
 		(pad "4" thru_hole oval
 			(at 0.000001 3.810001 90)
-			(size 2.3 3.2)
+			(size 1.7 3.2)
 			(drill 0.8
 				(offset 0 -0.4)
@@
 			(layers "*.Cu" "*.Mask")
 			(remove_unused_layers no)
+			(net 3 "+4V")
+			(pinfunction "BAT")
+			(pintype "power_in")
 		)
 		(model "${KIPRJMOD}/lib/lolin32/lolin32.step"
@@
 			(at -2.54 -0.000001)
 			(size 3.5 2)
-			(drill oval 1.8 0.8)
+			(drill oval 1.8 0.8
+				(offset 0 -0.3)
+			)
 			(layers "*.Cu" "*.Mask")
 			(remove_unused_layers no)
@@
 			(at 2.54 0.000001)
 			(size 3.5 2)
-			(drill oval 1.8 0.8)
+			(drill oval 1.8 0.8
+				(offset 0 0.3)
+			)
 			(layers "*.Cu" "*.Mask")
 			(remove_unused_layers no)
@@
 		(pad "2" thru_hole oval
 			(at 0 0 270)
-			(size 2.5 3.5)
+			(size 2 3)
 			(drill 0.8)
 			(layers "*.Cu" "*.Mask")
@@
 	)
 	(gr_text "April 26\n#288"
-		(at 127 62.8 45)
+		(at 127.22453 62.5663 45)
 		(layer "B.Cu" knockout)
 		(effects
@@
 	)
 	(gr_text "+"
-		(at 89.25 86.5 -90)
+		(at 89.2 86.4 -90)
 		(layer "B.Cu" knockout)
 		(effects
@@
 	)
 	(segment
-		(start 81 97.009686)
-		(end 75.599696 91.609382)
+		(start 66.662943 67.587057)
+		(end 66.662943 68.813336)
 		(width 1)
 		(layer "B.Cu")
@@
 	)
 	(segment
-		(start 66.662943 67.587057)
-		(end 66.662943 68.813336)
+		(start 140.403792 100.894497)
+		(end 138.283774 100.894497)
 		(width 1)
 		(layer "B.Cu")
@@
 	)
 	(segment
-		(start 140.403792 100.894497)
-		(end 138.283774 100.894497)
+		(start 138.134398 100.745121)
+		(end 133.02 100.745121)
 		(width 1)
 		(layer "B.Cu")
@@
 	)
 	(segment
-		(start 85.589541 113.739999)
-		(end 81 109.150458)
+		(start 136.713926 111.45)
+		(end 128.100357 111.45)
 		(width 1)
 		(layer "B.Cu")
@@
 	)
 	(segment
-		(start 138.134398 100.745121)
-		(end 133.02 100.745121)
+		(start 128.100357 111.45)
+		(end 125.810358 113.739999)
 		(width 1)
 		(layer "B.Cu")
@@
 	)
 	(segment
+		(start 119.76 137.5)
+		(end 123.76 133.5)
+		(width 1)
+		(layer "B.Cu")
+		(net 2)
+	)
+	(segment
 		(start 118.5 119.25)
 		(end 119.415076 118.334924)
@@
 	)
 	(segment
+		(start 81 109.150458)
+		(end 81 97.009686)
+		(width 1)
+		(layer "B.Cu")
+		(net 2)
+	)
+	(segment
 		(start 66.662943 68.813336)
 		(end 74.049608 76.200001)
@@
 	)
 	(segment
+		(start 136.972392 111.191534)
+		(end 136.713926 111.45)
+		(width 1)
+		(layer "B.Cu")
+		(net 2)
+	)
+	(segment
+		(start 123.76 133.5)
+		(end 123.76 131)
+		(width 1)
+		(layer "B.Cu")
+		(net 2)
+	)
+	(segment
 		(start 133.307107 96.294497)
 		(end 140.597746 96.294497)
@@
 	)
 	(segment
+		(start 85.589541 113.739999)
+		(end 81 109.150458)
+		(width 1)
+		(layer "B.Cu")
+		(net 2)
+	)
+	(segment
 		(start 122.36 96.580169)
 		(end 122.36 94.6)
@@
 	)
 	(segment
-		(start 136.713926 111.45)
-		(end 128.100357 111.45)
-		(width 1)
-		(layer "B.Cu")
-		(net 2)
-	)
-	(segment
 		(start 95.6 80.1)
 		(end 95.6 97.043857)
@@
 	)
 	(segment
-		(start 125.810358 113.739999)
-		(end 85.589541 113.739999)
-		(width 1)
-		(layer "B.Cu")
-		(net 2)
-	)
-	(segment
 		(start 143.875685 106.875685)
 		(end 141.288241 106.875685)
@@
 	)
 	(segment
+		(start 81 97.009686)
+		(end 75.599696 91.609382)
+		(width 1)
+		(layer "B.Cu")
+		(net 2)
+	)
+	(segment
 		(start 95.6 97.043857)
 		(end 85.66 106.983857)
@@
 	)
 	(segment
-		(start 128.100357 111.45)
-		(end 125.810358 113.739999)
+		(start 106.5 137.5)
+		(end 119.76 137.5)
 		(width 1)
 		(layer "B.Cu")
@@
 	)
 	(segment
-		(start 131.457244 118.334924)
-		(end 134.304668 115.4875)
+		(start 125.810358 113.739999)
+		(end 85.589541 113.739999)
 		(width 1)
 		(layer "B.Cu")
@@
 	)
 	(segment
-		(start 74.049608 76.200001)
-		(end 91.700001 76.200001)
+		(start 131.457244 118.334924)
+		(end 134.304668 115.4875)
 		(width 1)
 		(layer "B.Cu")
@@
 	)
 	(segment
-		(start 81 109.150458)
-		(end 81 97.009686)
+		(start 74.049608 76.200001)
+		(end 91.700001 76.200001)
 		(width 1)
 		(layer "B.Cu")
@@
 	)
 	(segment
-		(start 136.972392 111.191534)
-		(end 136.713926 111.45)
-		(width 1)
-		(layer "B.Cu")
-		(net 2)
-	)
-	(segment
 		(start 85.66 106.983857)
 		(end 85.66 108.14)
@@
 	)
 	(segment
-		(start 78.83 112.58)
-		(end 78.83 105.97)
+		(start 88.5 115.54)
+		(end 90.96 118)
 		(width 1)
 		(layer "B.Cu")
@@
 	)
 	(segment
-		(start 88.5 115.54)
-		(end 90.96 118)
+		(start 78.83 105.97)
+		(end 78.83 112.58)
 		(width 1)
 		(layer "B.Cu")
@@
 	)
 	(segment
+		(start 78.83 102.08)
+		(end 78.83 105.97)
+		(width 1)
+		(layer "B.Cu")
+		(net 3)
+	)
+	(segment
 		(start 88.5 115.54)
 		(end 81.79 115.54)
@@
 	)
 	(segment
-		(start 78.83 102.08)
-		(end 78.83 105.97)
-		(width 1)
-		(layer "B.Cu")
-		(net 3)
-	)
-	(segment
 		(start 119.82 88)
 		(end 119.82 94.6)
@@
 	)
 	(segment
-		(start 105 74.68)
-		(end 105 102.8)
+		(start 95.82 106.04)
+		(end 95.82 108.14)
 		(width 0.6)
 		(layer "B.Cu")
@@
 	)
 	(segment
-		(start 105 102.8)
-		(end 102.26 105.54)
+		(start 96.66 105.2)
+		(end 95.82 106.04)
 		(width 0.6)
 		(layer "B.Cu")
@@
 	)
 	(segment
-		(start 104.973833 62.973833)
-		(end 104.973833 74.493833)
+		(start 105 74.68)
+		(end 105 102.8)
 		(width 0.6)
 		(layer "B.Cu")
@@
 	)
 	(segment
-		(start 95.82 106.04)
-		(end 95.82 108.14)
+		(start 105 102.8)
+		(end 102.6 105.2)
 		(width 0.6)
 		(layer "B.Cu")
@@
 	)
 	(segment
-		(start 102.26 105.54)
-		(end 96.32 105.54)
+		(start 104.973833 62.973833)
+		(end 104.973833 74.493833)
 		(width 0.6)
 		(layer "B.Cu")
@@
 	)
 	(segment
-		(start 100 58)
-		(end 104.973833 62.973833)
+		(start 102.6 105.2)
+		(end 96.66 105.2)
 		(width 0.6)
 		(layer "B.Cu")
@@
 	)
 	(segment
-		(start 96.32 105.54)
-		(end 95.82 106.04)
+		(start 100 58)
+		(end 104.973833 62.973833)
 		(width 0.6)
 		(layer "B.Cu")
@@
 	)
 	(segment
-		(start 83.71 106.671115)
-		(end 83.71 109.597716)
+		(start 91.9 79.5)
+		(end 93.85 81.45)
 		(width 0.6)
 		(layer "B.Cu")
@@
 	)
 	(segment
-		(start 83.71 109.597716)
-		(end 84.852284 110.74)
+		(start 90.24 110.74)
+		(end 90.74 110.24)
 		(width 0.6)
 		(layer "B.Cu")
@@
 	)
 	(segment
-		(start 91.25 79.5)
-		(end 93.85 82.1)
+		(start 83.71 106.671115)
+		(end 83.71 109.597716)
 		(width 0.6)
 		(layer "B.Cu")
@@
 	)
 	(segment
-		(start 90.24 110.74)
-		(end 90.74 110.24)
+		(start 93.85 81.45)
+		(end 93.85 96.531115)
 		(width 0.6)
 		(layer "B.Cu")
@@
 	)
 	(segment
-		(start 90.74 110.24)
-		(end 90.74 108.14)
+		(start 91.25 79.5)
+		(end 91.9 79.5)
 		(width 0.6)
 		(layer "B.Cu")
@@
 	)
 	(segment
-		(start 93.85 82.1)
-		(end 93.85 96.531115)
+		(start 93.85 96.531115)
+		(end 83.71 106.671115)
 		(width 0.6)
 		(layer "B.Cu")
@@
 	)
 	(segment
-		(start 93.85 96.531115)
-		(end 83.71 106.671115)
+		(start 90.74 110.24)
+		(end 90.74 108.14)
+		(width 0.6)
+		(layer "B.Cu")
+		(net 23)
+	)
+	(segment
+		(start 83.71 109.597716)
+		(end 84.852284 110.74)
 		(width 0.6)
 		(layer "B.Cu")
