File: sandwichlamp.kicad_sch (KiCad schematic)
At the start: 27 parts, among them J1 Pole1, J2 Pole2, J3 Pole3, J4 12V Enable, J5 HLK-LD2410C, J6 Conn_01x02, J7 Conn_01x03, SW1 Rader Power, SW3 POWER, U1 magnetic-charger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

Commit message: Run DRC
Connections:
- net +4V: now also U7.37 (BAT)
Changed lines of the file:
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@@
 		(pin "25"
+		)
+		(pin "37"
 		)
 		(instances
@@
 					(unit 1)
 				)
+			)
+		)
+	)
+	(symbol
+		(lib_id "power:+4V")
+		(at 130.81 100.33 90)
+		(unit 1)
+		(exclude_from_sim no)
+		(in_bom yes)
+		(on_board yes)
+		(dnp no)
+		(fields_autoplaced yes)
+		(property "Reference" "#PWR015"
+			(at 134.62 100.33 0)
+			(effects
+				(font
+					(size 1.27 1.27)
+				)
+				(hide yes)
+			)
+		)
+		(property "Value" "+4V"
+			(at 127 100.3299 90)
+			(effects
+				(font
+					(size 1.27 1.27)
+				)
+				(justify left)
+			)
+		)
+		(property "Footprint" ""
+			(at 130.81 100.33 0)
+			(effects
+				(font
+					(size 1.27 1.27)
+				)
+				(hide yes)
+			)
+		)
+		(property "Datasheet" ""
+			(at 130.81 100.33 0)
+			(effects
+				(font
+					(size 1.27 1.27)
+				)
+				(hide yes)
+			)
+		)
+		(property "Description" "Power symbol creates a global label with name \"+4V\""
+			(at 130.81 100.33 0)
+			(effects
+				(font
+					(size 1.27 1.27)
+				)
+				(hide yes)
+			)
+		)
+		(pin "1"
+		)
+		(instances
+			(project "sandwichlamp"
+				(path "/e0ec050d-3d79-41e4-bfa7-38c68df5e8aa"
+					(reference "#PWR015")
+					(unit 1)
+				)

Commit message: Reverse the polarity of the SMD Battery Connector
Connections:
- net GND: now also BT1.1 (-); no longer BT1.2 (-)
- net VBAT: now also BT1.2 (+); no longer BT1.1 (+)
Changed lines of the file:
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@@
 	)
 	(symbol
+		(lib_name "Battery_Cell_1")
 		(lib_id "Device:Battery_Cell")
 		(at 34.29 78.74 0)
